File: 60mmledmatrixesp32c3.kicad_sch (KiCad schematic)
At the start: 10 parts, among them J1 CUI_PJ-002BH-SMT-TR, J2 Grounded Mounting Hole, J3 Grounded Mounting Hole, J4 Grounded Mounting Hole, J5 Grounded Mounting Hole, U7 ESP32-C3_SUPERMINI

Commit message: Added PDF schema
Other:
- company: (none) -> stig@sdm.nz
- title: (none) -> esp32c3 Led Matrix 6x8x8
Changed lines of the file:
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@@
 	(generator_version "8.0")
 	(paper "A4")
+	(title_block
+		(title "esp32c3 Led Matrix 6x8x8")
+		(company "stig@sdm.nz")
+		(comment 1 "BSD 2-Clause License")
+	)
 	(junction
 		(at 170.18 57.15)
