File: matrix1.kicad_sch (KiCad schematic)
At the start: 5 parts, among them U5 MAX7221CWG+T

Commit message: Added PDF schema
Other:
- title: (none) -> esp32c3 Led Matrix 6x8x8 - Matrix Schema
- moved on the sheet: C10, C9, D5, R5, U5
